Commit message: Add files via upload

File: src/my_bot/description/agv.urdf.xacro (robot description, xacro)
@@ -208,5 +208,5 @@
         <parent link="base_link"/>
         <child link="camera_link"/>
-        <origin xyz="0.6 0 0.2" rpy="0 0 0"/>
+        <origin xyz="0.6 0 0.2" rpy="0 ${pi/6} 0"/>
   </joint>
   <link name="camera_link">

Commit message: Update Line Following and route tracking

File: src/my_bot/description/agv.urdf.xacro (robot description, xacro)
@@ -208,5 +208,5 @@
         <parent link="base_link"/>
         <child link="camera_link"/>
-        <origin xyz="0.6 0 0.2" rpy="0 ${pi/6} 0"/>
+        <origin xyz="0.6 0 0.2" rpy="0 ${pi/2} 0"/>
   </joint>
   <link name="camera_link">
